Commit message: Added dae and reduced properties in global namespace.

File: urdf/sick_lms1xx.urdf.xacro (robot description, xacro)
@@ -26,27 +26,19 @@
 -->
 <robot xmlns:xacro="http://ros.org/wiki/xacro">
-  <xacro:property name="laser_x" value="0.105" />
-  <xacro:property name="laser_y" value="0.102" />
-  <xacro:property name="laser_z" value="0.152" />
-  <xacro:property name="laser_mass" value="1.1" />
-  <xacro:macro name="box_inertial" params="x y z mass">
-    <inertial>
-      <mass value="${mass}" />
-      <origin xyz="0 0 0" />
-      <inertia ixx="${0.0833333 * mass * (y*y + z*z)}" ixy="0.0" ixz="0.0"
-        iyy="${0.0833333 * mass * (x*x + z*z)}" iyz="0.0"
-        izz="${0.0833333 * mass * (x*x + y*y)}" />
-    </inertial>
-  </xacro:macro>
   <xacro:macro name="sick_lms1xx" params="prefix topic">
     <link name="${prefix}_laser">
-      <xacro:box_inertial x="${laser_x}" y="${laser_y}" z="${laser_z}" mass="${laser_mass}" />
+      <inertial>
+        <mass value="1.1" />
+        <origin xyz="0 0 0" />
+        <inertia ixx="${0.0833333 * mass * (0.102*0.102 + 0.152*0.152)}" ixy="0.0" ixz="0.0"
+          iyy="${0.0833333 * 1.1 * (0.105*0.105 + 0.152*0.152)}" iyz="0.0"
+          izz="${0.0833333 * 1.1 * (0.105*0.105 + 0.102*0.102)}" />
+      </inertial>
       <visual>
         <origin xyz="0 0 0" rpy="0 0 0" />
         <geometry>
           <!-- Origin of this mesh is the focal point of the LIDAR. -->
-          <mesh filename="package://lms1xx/meshes/sick-lms1xx.stl" />
+          <mesh filename="package://lms1xx/meshes/sick-lms1xx.dae" />
         </geometry>
-        <material name="light_grey" />
       </visual>
       <collision>
@@ -58,5 +50,4 @@
     </link>
     <gazebo reference="${prefix}_laser">
-      <material>Gazebo/Grey</material>
       <turnGravityOff>true</turnGravityOff>
       <sensor type="ray" name="${prefix}_laser">
